Commit message: Major updates to Ch::ROS

File: data/robot/r2d2/r2d2.urdf (robot description, URDF)
Before this commit: robot physics, 16 links, 15 joints
Links:
- link left_gripper: geometry collision mesh filename=./meshes/l_finger.dae; visual mesh filename=./meshes/l_finger.dae
- link left_tip: geometry collision mesh filename=./meshes/l_finger_tip.dae; visual mesh filename=./meshes/l_finger_tip.dae
- link right_gripper: geometry collision mesh filename=./meshes/l_finger.dae; visual mesh filename=./meshes/l_finger.dae
- link right_tip: geometry collision mesh filename=./meshes/l_finger_tip.dae; visual mesh filename=./meshes/l_finger_tip.dae

Commit message: Reverted r2d2

File: data/robot/r2d2/r2d2.urdf (robot description, URDF)
Before this commit: robot physics, 16 links, 15 joints
Links:
- link left_gripper: geometry collision mesh filename=meshes/l_finger.dae; visual mesh filename=meshes/l_finger.dae
- link left_tip: geometry collision mesh filename=meshes/l_finger_tip.dae; visual mesh filename=meshes/l_finger_tip.dae
- link right_gripper: geometry collision mesh filename=meshes/l_finger.dae; visual mesh filename=meshes/l_finger.dae
- link right_tip: geometry collision mesh filename=meshes/l_finger_tip.dae; visual mesh filename=meshes/l_finger_tip.dae
